Commit message: Added nav2 params

File: config/rocker.urdf (robot description, URDF)
Before this commit: robot Rocker, 18 links, 17 joints
Links:
- removed link Chassis-v2
- added link base_link
- added link imu_link
Joints:
- removed joint Chassis-v2_Rigid-1
- removed joint Chassis-v2_Rigid-17
- removed joint Chassis-v2_Rigid-2
- added joint base_link_IMU: type fixed, parent base_link, child imu_link, origin xyz=0.0 0.0 0.0 rpy=0.0 0.0 0.0
- added joint base_link_Rigid-1: type fixed, parent base_link, child Righ-Rocker-v2, origin xyz=0.020280175196496372 0.02899987748248961 0.0933999999999999 rpy=0.0 -0.0 0.0, axis 0.0 0.0 1.0
- added joint base_link_Rigid-17: type fixed, parent base_link, child Camera-v6, origin xyz=-0.1693998248000423 0.029001023390823395 -5.684341886080802e-16 rpy=6.041271265845756e-06 1.5707963267948966 0
- added joint base_link_Rigid-2: type fixed, parent base_link, child Left-Rocker-v2, origin xyz=0.020280175196496372 0.02899987748248961 -0.09340000000000032 rpy=0.0 -0.0 0.0, axis 0.0 0.0 1.0
