Commit message: Updated namespace consistent

File: config/mini.urdf (robot description, URDF)
Before this commit: robot mini_clean, 0 links, 0 joints
Links:
- added link ${ns_prefix}base_link
- added link ${ns_prefix}front_left_wheel_link
- added link ${ns_prefix}front_right_wheel_link
- added link ${ns_prefix}left_cam
- added link ${ns_prefix}left_ir_sensor
- added link ${ns_prefix}rear_left_wheel_link
- added link ${ns_prefix}rear_right_wheel_link
- added link ${ns_prefix}right_cam
- added link ${ns_prefix}right_ir_sensor
Joints:
- added joint Front_Left_Wheel: type continuous, parent ${ns_prefix}base_link, child ${ns_prefix}front_left_wheel_link, origin xyz=-0.0582 -0.039 0.00965 rpy=1.5707963267948963 0.0 3.141592653589793, axis 0.0 1.0 0.0
- added joint Front_Right_Wheel: type continuous, parent ${ns_prefix}base_link, child ${ns_prefix}front_right_wheel_link, origin xyz=0.0582 -0.039 0.00965 rpy=1.5707963267948966 0.0 0.0, axis 0.0 -1.0 0.0
- added joint Left_Cam: type fixed, parent ${ns_prefix}base_link, child ${ns_prefix}left_cam, origin xyz=0.039709 -0.066324 0.027 rpy=1.5707963267948968 0.0 -0.4363323129987227
- added joint Rear_Left_Wheel: type continuous, parent ${ns_prefix}base_link, child ${ns_prefix}rear_left_wheel_link, origin xyz=-0.0582 0.039 0.00965 rpy=1.5707963267948966 0.0 3.141592653589793, axis 0.0 1.0 0.0
- added joint Rear_Right_Wheel: type continuous, parent ${ns_prefix}base_link, child ${ns_prefix}rear_right_wheel_link, origin xyz=0.0582 0.039 0.00965 rpy=1.5707963267948963 0.0 0.0, axis 0.0 -1.0 0.0
- added joint Right_Cam: type fixed, parent ${ns_prefix}base_link, child ${ns_prefix}right_cam, origin xyz=-0.03970 -0.066324 0.027 rpy=-1.5707963267948966 0.0 -2.705260340591013
- added joint base_link_Left-Avoidance-Sensor: type fixed, parent ${ns_prefix}base_link, child ${ns_prefix}left_ir_sensor, origin xyz=0.05399999999999989 0.06249999999999997 0.020870000000000007 rpy=0.0 0.0 0.0
- added joint base_link_Right-Avoidance-Sensor: type fixed, parent ${ns_prefix}base_link, child ${ns_prefix}right_ir_sensor, origin xyz=-0.05400000000000011 0.06250000000000001 0.020870000000000007 rpy=0.0 0.0 0.0

Commit message: Fixed joint_state_broadcaster_spawner and mecanum_controller_spawner

File: config/mini.urdf (robot description, URDF)
Before this commit: robot Mini, 9 links, 8 joints
Joints:
- joint Front_Left_Wheel: axis 0.0 1.0 0.0 -> 1.0 0.0 0.0
- joint Front_Right_Wheel: axis 0.0 -1.0 0.0 -> -1.0 0.0 0.0
- joint Rear_Left_Wheel: axis 0.0 1.0 0.0 -> 1.0 0.0 0.0
- joint Rear_Right_Wheel: axis 0.0 -1.0 0.0 -> -1.0 0.0 0.0

Commit message: clean up

File: config/mini.urdf (robot description, URDF)
Before this commit: robot Mini, 11 links, 10 joints
Links:
- removed link ${ns_prefix}left_cam
- removed link ${ns_prefix}left_ir_sensor
- removed link ${ns_prefix}right_cam
- removed link ${ns_prefix}right_ir_sensor
- removed link ${ns_prefix}uwb
Joints:
- removed joint Left_Cam
- removed joint Right_Cam
- removed joint base_link_Left_Avoidance_Sensor
- removed joint base_link_Right_Avoidance_Sensor
- removed joint base_link_UWB

Commit message: Updated

File: config/mini.urdf (robot description, URDF)
Before this commit: robot Mini, 6 links, 5 joints
Links:
- removed link ${ns_prefix}imu
- added link ${ns_prefix}imu_link
Joints:
- joint base_link_IMU: child ${ns_prefix}imu -> ${ns_prefix}imu_link

Commit message: Updated

File: config/mini.urdf (robot description, URDF)
Before this commit: robot Mini, 6 links, 5 joints
Links:
- removed link ${ns_prefix}imu_link
- added link ${ns_prefix}imu
- added link ${ns_prefix}left_cam
- added link ${ns_prefix}right_cam
- added link ${ns_prefix}uwb
Joints:
- added joint Left_Cam: type fixed, parent ${ns_prefix}base_link, child ${ns_prefix}left_cam, origin xyz=0.066324 0.039709 0.027 rpy=1.5707963267948968 0.0 1.134464013796174
- added joint Right_Cam: type fixed, parent ${ns_prefix}base_link, child ${ns_prefix}right_cam, origin xyz=0.066324 -0.0397 0.027 rpy=-1.5707963267948966 0.0 -1.1344640137961166
- added joint base_link_UWB: type fixed, parent ${ns_prefix}base_link, child ${ns_prefix}uwb, origin xyz=0.0 0.0 0.0 rpy=0.0 0.0 0.0
- joint base_link_IMU: child ${ns_prefix}imu_link -> ${ns_prefix}imu
